Commit message: Horizontal arc8

File: components/arm/elite_arm.urdf.xacro (robot description, xacro)
@@ -22,5 +22,5 @@
                 link_inertials_parameters_file="$(arg link_inertials_params_file)"
             >
-                <origin xyz="0.133 0.0 0.416" rpy="0.0 0.0 -1.5708" />
+                <origin xyz="0.133 0.0 0.416" rpy="0.0 0.0 1.5708" />  <!-- +90 deg like ur_arm.urdf.xacro (real mount, checked 2026-09-29) -->
             </xacro:elite_robot>
             <!-- If both Elite Arm and Simulation is used -->

File: components/arm/ur_arm.urdf.xacro (robot description, xacro)
@@ -39,5 +39,8 @@
                 >
                 <!-- position robot in the world -->
-                <origin xyz="0.133 0.0 0.416" rpy="0.0 0.0 -1.5708" />
+                <!-- yaw +90 deg: checked on the real robot 2026-09-29 (with -90 the arm pointed to the
+                     NEOBOTIX side in RViz / TF while the real arm points away from it, towards
+                     the robot's -x; LiDAR and base frames were correct) -->
+                <origin xyz="0.133 0.0 0.416" rpy="0.0 0.0 1.5708" />
             </xacro:ur_robot>
             <!-- If both UR Arm and Simulation is used -->

File: components/arm/wrist_camera_mount.urdf.xacro (robot description, xacro)
@@ -38,4 +38,10 @@
             <!-- Include wrist camera -->
             <xacro:include filename="$(find steve_simulation)/components/cameras/wrist_d405.urdf.xacro"/>
-            <xacro:wrist_d405 parent="dummy_end_effector" use_gazebo="$(arg use_gazebo)"/>
+            <!-- real robot: wrist D415 looks along the tool axis (no bracket tilt) -->
+            <xacro:if value="$(arg use_gazebo)">
+              <xacro:wrist_d405 parent="dummy_end_effector" use_gazebo="$(arg use_gazebo)"/>
+            </xacro:if>
+            <xacro:unless value="$(arg use_gazebo)">
+              <xacro:wrist_d405 parent="dummy_end_effector" use_gazebo="$(arg use_gazebo)" tilt="0.0"/>
+            </xacro:unless>
 </robot>

File: components/cameras/wrist_d405.urdf.xacro (robot description, xacro)
@@ -1,5 +1,5 @@
 <?xml version="1.0"?>
 <robot xmlns:xacro="http://ros.org/wiki/xacro">
-<xacro:macro name="wrist_d405" params="parent use_gazebo">
+<xacro:macro name="wrist_d405" params="parent use_gazebo tilt:=${pi/12}">
 <material name="grey">
   <color rgba="0.5 0.5 0.5 1"/>
@@ -35,5 +35,7 @@
   <child link="wrist_camera_link"/>
   <!-- mount is angled 15° - pi/12 -->
-  <origin xyz="0.079 0.0 0.047" rpy="0.0 ${-pi/2+pi/12} ${pi}"/>
+  <!-- tilt: camera axis vs. the tool axis. D405 bracket (Gazebo): 15 deg; the real wrist D415 looks
+       along the tool axis (measured with the table plane, 2026-09-29: 13.6 deg error with 15 deg) -->
+  <origin xyz="0.079 0.0 0.047" rpy="0.0 ${-pi/2+tilt} ${pi}"/>
 </joint>
 <link name="wrist_camera_link">

File: components/dynamixel/dynamixel_bracket_fr12_h101.urdf.xacro (robot description, xacro)
@@ -1,5 +1,5 @@
 <?xml version="1.0"?>
 <robot xmlns:xacro="http://www.ros.org/wiki/xacro">
-  <xacro:macro name="dynamixel_bracket_dynamixel_bracket_FR12_H101" params="parent name *origin">
+  <xacro:macro name="dynamixel_bracket_dynamixel_bracket_FR12_H101" params="parent name *origin visual_xyz:='0 0 0' visual_rpy:='0 0 0'">
     <joint name="${name}_joint" type="fixed" >
       <xacro:insert_block name="origin" />
@@ -14,5 +14,5 @@
       </inertial>
       <visual>
-        <origin xyz="0 0 0" rpy="0 0 0" />
+        <origin xyz="${visual_xyz}" rpy="${visual_rpy}" />
         <geometry>
           <mesh filename="package://steve_simulation/robots/mmo_700/meshes/cameras/dynamixel/dynamixel_bracket_fr12_h101.dae" scale="0.001 0.001 0.001" />
@@ -20,5 +20,5 @@
       </visual>
       <collision>
-        <origin xyz="0 0 0" rpy="0 0 0" />
+        <origin xyz="${visual_xyz}" rpy="${visual_rpy}" />
         <geometry>
           <mesh filename="package://steve_simulation/robots/mmo_700/meshes/cameras/dynamixel/dynamixel_bracket_fr12_h101_convex_hull.dae" scale="0.001 0.001 0.001" />

File: components/dynamixel/dynamixel_motor_xl-430.urdf.xacro (robot description, xacro)
@@ -4,5 +4,5 @@
   <xacro:include filename="$(find steve_simulation)/components/dynamixel/dynamixel_motor_xl-430.transmission.xacro" />
   <xacro:property name="M_PI" value="3.1415926535897931" />
-  <xacro:macro name="dynamixel_motor_XL-430" params="parent name *origin motor_direction position_offset">
+  <xacro:macro name="dynamixel_motor_XL-430" params="parent name *origin motor_direction position_offset visual_xyz:='0 0 0' visual_rpy:='0 ${pi/2} 0'">
     <joint name="${name}_base_joint" type="fixed" >
       <xacro:insert_block name="origin" />
@@ -17,5 +17,5 @@
       </inertial>
       <visual>
-        <origin xyz="0 0 0.0" rpy="0 ${pi/2} 0" />
+        <origin xyz="${visual_xyz}" rpy="${visual_rpy}" />
         <geometry>
           <mesh filename="package://steve_simulation/robots/mmo_700/meshes/cameras/dynamixel/dynamixel_motor_xl-430.dae" scale="0.001 0.001 0.001" />
@@ -23,5 +23,5 @@
       </visual>
       <collision>
-        <origin xyz="0 0 0.0" rpy="0 ${M_PI/2} 0" />
+        <origin xyz="${visual_xyz}" rpy="${visual_rpy}" />
         <geometry>
           <mesh filename="package://steve_simulation/robots/mmo_700/meshes/cameras/dynamixel/dynamixel_motor_xl-430_convex_hull.dae" scale="0.001 0.001 0.001" />

File: components/dynamixel/steve_pan_tilt.xacro (robot description, xacro)
@@ -4,19 +4,25 @@
   <xacro:include filename="$(find steve_simulation)/components/dynamixel/dynamixel_bracket_fr12_h101.urdf.xacro" />
   <xacro:arg name="grasp_link_offset" default="0.11"/>
-+  <xacro:macro name="steve_pan_tilt" params="parent name">
+  <!-- Mesh visual origins reproduce the mesh placement of the MuJoCo model
+       (steve_wbc/models/mmo_700_wbc.xml); link/joint frames are unchanged. -->
+  <xacro:macro name="steve_pan_tilt" params="parent name">
     <!-- Pan motor -->
-    <xacro:dynamixel_motor_XL-430 name="${name}_tilt_motor" parent="${parent}" motor_direction="-1" position_offset="0.065">
+    <xacro:dynamixel_motor_XL-430 name="${name}_tilt_motor" parent="${parent}" motor_direction="-1" position_offset="0.065"
+                                 visual_rpy="0 0 0">
       <origin xyz="0.0 0.0 0.4855" rpy="${-3*pi/2} 0 ${pi/2}" />
     </xacro:dynamixel_motor_XL-430>
     <!-- Pan bracket -->
-    <xacro:dynamixel_bracket_dynamixel_bracket_FR12_H101 name="${name}_tilt_bracket" parent="${name}_tilt_motor_link">
+    <xacro:dynamixel_bracket_dynamixel_bracket_FR12_H101 name="${name}_tilt_bracket" parent="${name}_tilt_motor_link"
+                                                  visual_rpy="${pi-0.065} 0 ${pi}">
       <origin xyz="0 0 0" rpy="${pi/2-0.065} 0 0" />
     </xacro:dynamixel_bracket_dynamixel_bracket_FR12_H101>
     <!-- Tilt motor -->
-    <xacro:dynamixel_motor_XL-430 name="${name}_pan_motor" parent="${name}_tilt_bracket_link" motor_direction="-1" position_offset="0.065">
+    <xacro:dynamixel_motor_XL-430 name="${name}_pan_motor" parent="${name}_tilt_bracket_link" motor_direction="-1" position_offset="0.065"
+                                 visual_xyz="-0.0041 0 0" visual_rpy="${pi} 0 ${-(pi-0.065)}">
       <origin xyz="0 0.0633 0" rpy="0 ${pi/2} 0" />
     </xacro:dynamixel_motor_XL-430>
     <!-- Tilt bracket -->
-    <xacro:dynamixel_bracket_dynamixel_bracket_FR12_H101 name="${name}_pan_bracket" parent="${name}_pan_motor_link">
+    <xacro:dynamixel_bracket_dynamixel_bracket_FR12_H101 name="${name}_pan_bracket" parent="${name}_pan_motor_link"
+                                                  visual_xyz="0.0041 0 0" visual_rpy="${pi-0.065} 0 -0.065">
       <origin xyz="0 0 0" rpy="${pi-0.065} 0 0" />
     </xacro:dynamixel_bracket_dynamixel_bracket_FR12_H101>

File: robots/mmo_700/mmo_700_processed.urdf (robot description, URDF)
Before this commit: robot mmo_700, 42 links, 41 joints
Joints:
- joint ur5ebase_joint: origin xyz=0.133 0.0 0.416 rpy=0.0 0.0 -1.5708 -> xyz=0.133 0.0 0.416 rpy=0.0 0.0 1.5708
